Commit message: 暂存调试版本吗

File: agribot_ws/src/agribot_simulation/urdf/agribot/agribot.gazebo.xacro (robot description, xacro)
@@ -8,7 +8,7 @@
     </gazebo>
     <gazebo reference="lf_wheel_link">
-        <mu1>1</mu1>
-        <mu2>1</mu2>
-        <kp>100000.0</kp>
+        <mu1>10</mu1>
+        <mu2>10</mu2>
+        <kp>100000000.0</kp>
         <kd>1.0</kd>
         <minDepth>0.001</minDepth>
@@ -16,7 +16,7 @@
     </gazebo>
     <gazebo reference="rf_wheel_link">
-        <mu1>1</mu1>
-        <mu2>1</mu2>
-        <kp>100000.0</kp>
+        <mu1>10</mu1>
+        <mu2>10</mu2>
+        <kp>100000000.0</kp>
         <kd>1.0</kd>
         <minDepth>0.001</minDepth>
@@ -24,7 +24,7 @@
     </gazebo>
     <gazebo reference="lb_wheel_link">
-        <mu1>1</mu1>
-        <mu2>1</mu2>
-        <kp>100000.0</kp>
+        <mu1>10</mu1>
+        <mu2>10</mu2>
+        <kp>100000000.0</kp>
         <kd>1.0</kd>
         <minDepth>0.001</minDepth>
@@ -32,7 +32,7 @@
     </gazebo>
     <gazebo reference="rb_wheel_link">
-        <mu1>1</mu1>
-        <mu2>1</mu2>
-        <kp>100000.0</kp>
+        <mu1>10</mu1>
+        <mu2>10</mu2>
+        <kp>100000000.0</kp>
         <kd>1.0</kd>
         <minDepth>0.001</minDepth>

File: agribot_ws/src/agribot_simulation/urdf/agribot/mini_4wd_robot.urdf (robot description, URDF)
Before this commit: robot mini_4wd_robot, 8 links, 7 joints
Links:
- added link base_footprint
Joints:
- added joint base_joint: type fixed, parent base_footprint, child base_link, origin xyz=0 0 0 rpy=0 0 0
