Commit message: 完成对twoworld和corn_lead_world的仿真实验数据测试

File: agribot_ws/install/diff_drive_robot/share/diff_drive_robot/urdf/agribot_diff_drive.gazebo.xacro (robot description, xacro)
@@ -1,52 +1 @@
-<?xml version="1.0"?>
-<robot xmlns:xacro="http://www.ros.org/wiki/xacro">
-  <!-- Gazebo-specific material and friction properties only -->
-  <!-- Diff drive is handled by gazebo_ros2_control -->
-  <!-- Chassis Gazebo properties -->
-  <gazebo reference="base_link">
-    <material>Gazebo/Blue</material>
-    <mu1>0.8</mu1>
-    <mu2>0.8</mu2>
-  </gazebo>
-  <!-- Controller Gazebo properties -->
-  <gazebo reference="controller_link">
-    <material>Gazebo/White</material>
-  </gazebo>
-  <!-- Wheel Gazebo properties -->
-  <gazebo reference="wheel_lf_link">
-    <material>Gazebo/Black</material>
-    <mu1>1.5</mu1>
-    <mu2>0.8</mu2>
-    <kp>1000000.0</kp>
-    <kd>10.0</kd>
-    <minDepth>0.001</minDepth>
-    <maxVel>5.0</maxVel>
-  </gazebo>
-  <gazebo reference="wheel_lb_link">
-    <material>Gazebo/Black</material>
-    <mu1>1.5</mu1>
-    <mu2>0.8</mu2>
-    <kp>1000000.0</kp>
-    <kd>10.0</kd>
-    <minDepth>0.001</minDepth>
-    <maxVel>5.0</maxVel>
-  </gazebo>
-  <gazebo reference="wheel_rf_link">
-    <material>Gazebo/Black</material>
-    <mu1>1.5</mu1>
-    <mu2>0.8</mu2>
-    <kp>1000000.0</kp>
-    <kd>10.0</kd>
-    <minDepth>0.001</minDepth>
-    <maxVel>5.0</maxVel>
-  </gazebo>
-  <gazebo reference="wheel_rb_link">
-    <material>Gazebo/Black</material>
-    <mu1>1.5</mu1>
-    <mu2>0.8</mu2>
-    <kp>1000000.0</kp>
-    <kd>10.0</kd>
-    <minDepth>0.001</minDepth>
-    <maxVel>5.0</maxVel>
-  </gazebo>
-</robot>
+/home/xkai/agribot/agribot_ws/src/diff_drive_robot/urdf/agribot_diff_drive.gazebo.xacro

File: agribot_ws/install/diff_drive_robot/share/diff_drive_robot/urdf/agribot_diff_drive.ros2_control.xacro (robot description, xacro)
@@ -1,73 +1 @@
-<?xml version="1.0"?>
-<robot xmlns:xacro="http://www.ros.org/wiki/xacro">
-    <xacro:macro name="agribot_ros2_control">
-        <ros2_control name="AgriBotGazeboSystem" type="system">
-            <hardware>
-                <plugin>gazebo_ros2_control/GazeboSystem</plugin>
-            </hardware>
-            <joint name="wheel_lf_joint">
-                <command_interface name="velocity">
-                    <param name="min">-10</param>
-                    <param name="max">10</param>
-                </command_interface>
-                <command_interface name="effort">
-                    <param name="min">-5</param>
-                    <param name="max">5</param>
-                </command_interface>
-                <state_interface name="position" />
-                <state_interface name="velocity" />
-                <state_interface name="effort" />
-            </joint>
-            <joint name="wheel_lb_joint">
-                <command_interface name="velocity">
-                    <param name="min">-10</param>
-                    <param name="max">10</param>
-                </command_interface>
-                <command_interface name="effort">
-                    <param name="min">-5</param>
-                    <param name="max">5</param>
-                </command_interface>
-                <state_interface name="position" />
-                <state_interface name="velocity" />
-                <state_interface name="effort" />
-            </joint>
-            <joint name="wheel_rf_joint">
-                <command_interface name="velocity">
-                    <param name="min">-10</param>
-                    <param name="max">10</param>
-                </command_interface>
-                <command_interface name="effort">
-                    <param name="min">-5</param>
-                    <param name="max">5</param>
-                </command_interface>
-                <state_interface name="position" />
-                <state_interface name="velocity" />
-                <state_interface name="effort" />
-            </joint>
-            <joint name="wheel_rb_joint">
-                <command_interface name="velocity">
-                    <param name="min">-10</param>
-                    <param name="max">10</param>
-                </command_interface>
-                <command_interface name="effort">
-                    <param name="min">-5</param>
-                    <param name="max">5</param>
-                </command_interface>
-                <state_interface name="position" />
-                <state_interface name="velocity" />
-                <state_interface name="effort" />
-            </joint>
-        </ros2_control>
-        <gazebo>
-            <plugin filename="libgazebo_ros2_control.so" name="gazebo_ros2_control">
-                <robot_param>robot_description</robot_param>
-                <robot_param_node>robot_state_publisher</robot_param_node>
-                <parameters>$(find diff_drive_robot)/config/agribot_ros2_controller.yaml</parameters>
-                <ros>
-                    <remapping>/agribot_diff_drive_controller/cmd_vel_unstamped:=/cmd_vel</remapping>
-                    <remapping>/agribot_diff_drive_controller/odom:=/odom</remapping>
-                </ros>
-            </plugin>
-        </gazebo>
-    </xacro:macro>
-</robot>
+/home/xkai/agribot/agribot_ws/src/diff_drive_robot/urdf/agribot_diff_drive.ros2_control.xacro

File: agribot_ws/install/diff_drive_robot/share/diff_drive_robot/urdf/agribot_diff_drive.urdf.xacro (robot description, xacro)
@@ -1,149 +1 @@
-<?xml version="1.0"?>
-<robot xmlns:xacro="http://www.ros.org/wiki/xacro" name="agribot_diff_drive">
-  <!-- Import materials -->
-  <xacro:include filename="$(find diff_drive_robot)/urdf/materials.xacro"/>
-  <!-- Import Gazebo configurations -->
-  <xacro:include filename="$(find diff_drive_robot)/urdf/agribot_diff_drive.gazebo.xacro"/>
-  <!-- Import ROS2 Control configurations -->
-  <xacro:include filename="$(find diff_drive_robot)/urdf/agribot_diff_drive.ros2_control.xacro"/>
-  <!-- Import IMU sensor -->
-  <xacro:include filename="$(find agribot_simulation)/urdf/agribot/sensors/imu.urdf.xacro" />
-  <!-- Import mid360 lidar -->
-  <xacro:include filename="$(find ros2_livox_simulation)/urdf/mid360.xacro" />
-  <!-- Robot dimensions (from agribot) -->
-  <xacro:property name="chassis_length" value="0.25"/>
-  <xacro:property name="chassis_width" value="0.20"/>
-  <xacro:property name="chassis_height" value="0.08"/>
-  <xacro:property name="chassis_mass" value="2.5"/>
-  <xacro:property name="wheel_radius" value="0.032"/>
-  <xacro:property name="wheel_thickness" value="0.02"/>
-  <xacro:property name="wheel_mass" value="0.2"/>
-  <!-- Wheel positions (from agribot) -->
-  <xacro:property name="wheel_offset_x_front" value="0.0789"/>
-  <xacro:property name="wheel_offset_x_rear" value="0.0930"/>
-  <xacro:property name="wheel_offset_y_left" value="0.0909"/>
-  <xacro:property name="wheel_offset_y_right" value="0.0907"/>
-  <xacro:property name="wheel_offset_z" value="-0.0363"/>
-  <!-- Base footprint link (ground projection) -->
-  <link name="base_footprint"/>
-  <!-- Joint from base_footprint to base_link -->
-  <joint name="base_joint" type="fixed">
-    <parent link="base_footprint"/>
-    <child link="base_link"/>
-    <origin xyz="0 0 ${wheel_radius - wheel_offset_z}" rpy="0 0 0"/>
-  </joint>
-  <!-- Base link (chassis) -->
-  <link name="base_link">
-    <!-- Visual uses agribot mesh for appearance -->
-    <visual>
-      <geometry>
-        <mesh filename="file://$(find agribot_simulation)/urdf/meshes/mini_4wd_robot_meshes/base_link.STL"/>
-      </geometry>
-      <material name="chassis_blue"/>
-      <origin xyz="0 0 0" rpy="0 0 0"/>
-    </visual>
-    <!-- Collision uses simple box geometry -->
-    <collision>
-      <geometry>
-        <box size="${chassis_length} ${chassis_width} ${chassis_height}"/>
-      </geometry>
-      <origin xyz="0 0 0" rpy="0 0 0"/>
-    </collision>
-    <inertial>
-      <mass value="${chassis_mass}"/>
-      <origin xyz="0 0 0" rpy="0 0 0"/>
-      <inertia
-        ixx="${chassis_mass / 12.0 * (chassis_width * chassis_width + chassis_height * chassis_height)}"
-        ixy="0.0"
-        ixz="0.0"
-        iyy="${chassis_mass / 12.0 * (chassis_length * chassis_length + chassis_height * chassis_height)}"
-        iyz="0.0"
-        izz="${chassis_mass / 12.0 * (chassis_length * chassis_length + chassis_width * chassis_width)}"/>
-    </inertial>
-  </link>
-  <!-- Controller link -->
-  <link name="controller_link">
-    <!-- Visual uses agribot mesh for appearance -->
-    <visual>
-      <geometry>
-        <mesh filename="file://$(find agribot_simulation)/urdf/meshes/mini_4wd_robot_meshes/controller_link.STL"/>
-      </geometry>
-      <material name="chassis_blue"/>
-      <origin xyz="0 0 0" rpy="0 0 0"/>
-    </visual>
-    <!-- Collision uses simple box geometry -->
-    <collision>
-      <geometry>
-        <box size="0.08 0.05 0.03"/>
-      </geometry>
-      <origin xyz="0 0 0" rpy="0 0 0"/>
-    </collision>
-    <inertial>
-      <mass value="0.7"/>
-      <origin xyz="0 0 0" rpy="0 0 0"/>
-      <inertia
-        ixx="8.75e-05"
-        ixy="0"
-        ixz="0"
-        iyy="1.46e-04"
-        iyz="0"
-        izz="2.04e-04"/>
-    </inertial>
-  </link>
-  <joint name="controller_joint" type="fixed">
-    <origin xyz="-0.0556343132168706 -0.0407821141826353 0.0519999999999999" rpy="0 0 0"/>
-    <parent link="base_link"/>
-    <child link="controller_link"/>
-    <axis xyz="0 0 0"/>
-  </joint>
-  <!-- Macro for creating wheels -->
-  <xacro:macro name="wheel" params="prefix x_reflect y_reflect x_offset y_offset">
-    <link name="wheel_${prefix}_link">
-      <!-- Visual uses agribot mesh for appearance -->
-      <visual>
-        <geometry>
-          <mesh filename="file://$(find agribot_simulation)/urdf/meshes/mini_4wd_robot_meshes/${prefix}_wheel_link.STL"/>
-        </geometry>
-        <material name="wheel_black"/>
-        <origin xyz="0 0 0" rpy="0 0 0"/>
-      </visual>
-      <!-- Collision uses simple cylinder geometry -->
-      <collision>
-        <geometry>
-          <cylinder radius="${wheel_radius}" length="${wheel_thickness}"/>
-        </geometry>
-        <origin xyz="0 0 0" rpy="${pi / 2.0} 0 0"/>
-      </collision>
-      <inertial>
-        <mass value="${wheel_mass}"/>
-        <origin xyz="0 0 0" rpy="0 0 0"/>
-        <inertia
-          ixx="${wheel_mass / 12.0 * (3 * wheel_radius * wheel_radius + wheel_thickness * wheel_thickness)}"
-          ixy="0.0"
-          ixz="0.0"
-          iyy="${wheel_mass * wheel_radius * wheel_radius / 2.0}"
-          iyz="0.0"
-          izz="${wheel_mass / 12.0 * (3 * wheel_radius * wheel_radius + wheel_thickness * wheel_thickness)}"/>
-      </inertial>
-    </link>
-    <joint name="wheel_${prefix}_joint" type="continuous">
-      <parent link="base_link"/>
-      <child link="wheel_${prefix}_link"/>
-      <origin xyz="${x_reflect * x_offset} ${y_reflect * y_offset} ${wheel_offset_z}" rpy="0 0 0"/>
-      <axis xyz="0 1 0"/>
-    </joint>
-  </xacro:macro>
-  <!-- Create four wheels -->
-  <xacro:wheel prefix="lf" x_reflect="1" y_reflect="1" x_offset="${wheel_offset_x_front}" y_offset="${wheel_offset_y_left}"/>
-  <xacro:wheel prefix="lb" x_reflect="-1" y_reflect="1" x_offset="${wheel_offset_x_rear}" y_offset="${wheel_offset_y_left}"/>
-  <xacro:wheel prefix="rf" x_reflect="1" y_reflect="-1" x_offset="${wheel_offset_x_front}" y_offset="${wheel_offset_y_right}"/>
-  <xacro:wheel prefix="rb" x_reflect="-1" y_reflect="-1" x_offset="${wheel_offset_x_rear}" y_offset="${wheel_offset_y_right}"/>
-  <!-- ROS2 Control -->
-  <xacro:agribot_ros2_control />
-  <!-- IMU sensor -->
-  <xacro:imu_xacro xyz="0 0 0" />
-  <!-- mid360 lidar -->
-  <xacro:mid360 name="livox" parent="base_link" topic="mid360">
-    <origin xyz="0.1 0 0.1" rpy="0 0 0" />
-  </xacro:mid360>
-</robot>
+/home/xkai/agribot/agribot_ws/src/diff_drive_robot/urdf/agribot_diff_drive.urdf.xacro

File: agribot_ws/install/diff_drive_robot/share/diff_drive_robot/urdf/materials.xacro (robot description, xacro)
@@ -1,11 +1 @@
-<?xml version="1.0"?>
-<robot xmlns:xacro="http://www.ros.org/wiki/xacro">
-  <!-- Chassis material - Blue -->
-  <material name="chassis_blue">
-    <color rgba="0.2 0.4 0.8 1.0"/>
-  </material>
-  <!-- Wheel material - Black -->
-  <material name="wheel_black">
-    <color rgba="0.1 0.1 0.1 1.0"/>
-  </material>
-</robot>
+/home/xkai/agribot/agribot_ws/src/diff_drive_robot/urdf/materials.xacro

File: agribot_ws/install/diff_drive_robot/share/diff_drive_robot/urdf/robot.gazebo.xacro (robot description, xacro)
@@ -1,69 +1 @@
-<?xml version="1.0"?>
-<robot xmlns:xacro="http://www.ros.org/wiki/xacro">
-  <!-- Gazebo plugin for differential drive -->
-  <gazebo>
-    <plugin name="diff_drive_controller" filename="libgazebo_ros_diff_drive.so">
-      <!-- Update rate -->
-      <update_rate>30</update_rate>
-      <!-- Wheel pairs -->
-      <num_wheel_pairs>2</num_wheel_pairs>
-      <!-- Left wheels (pair 0) -->
-      <left_joint>wheel_front_left_joint</left_joint>
-      <left_joint>wheel_rear_left_joint</left_joint>
-      <!-- Right wheels (pair 0) -->
-      <right_joint>wheel_front_right_joint</right_joint>
-      <right_joint>wheel_rear_right_joint</right_joint>
-      <!-- Kinematics -->
-      <wheel_separation>0.24</wheel_separation>
-      <wheel_radius>0.05</wheel_radius>
-      <!-- Limits -->
-      <max_wheel_torque>10</max_wheel_torque>
-      <max_wheel_acceleration>1.0</max_wheel_acceleration>
-      <!-- Output -->
-      <odometry_frame>odom</odometry_frame>
-      <robot_base_frame>base_footprint</robot_base_frame>
-      <!-- Odometry publishing -->
-      <publish_odom>true</publish_odom>
-      <publish_odom_tf>true</publish_odom_tf>
-      <publish_wheel_tf>true</publish_wheel_tf>
-      <!-- Topic -->
-      <command_topic>cmd_vel</command_topic>
-      <odometry_topic>odom</odometry_topic>
-    </plugin>
-  </gazebo>
-  <!-- Chassis Gazebo properties -->
-  <gazebo reference="base_link">
-    <material>Gazebo/Blue</material>
-    <mu1>0.5</mu1>
-    <mu2>0.5</mu2>
-  </gazebo>
-  <!-- Wheel Gazebo properties -->
-  <gazebo reference="wheel_front_left_link">
-    <material>Gazebo/Black</material>
-    <mu1>1.0</mu1>
-    <mu2>1.0</mu2>
-    <kp>1000000.0</kp>
-    <kd>100.0</kd>
-  </gazebo>
-  <gazebo reference="wheel_rear_left_link">
-    <material>Gazebo/Black</material>
-    <mu1>1.0</mu1>
-    <mu2>1.0</mu2>
-    <kp>1000000.0</kp>
-    <kd>100.0</kd>
-  </gazebo>
-  <gazebo reference="wheel_front_right_link">
-    <material>Gazebo/Black</material>
-    <mu1>1.0</mu1>
-    <mu2>1.0</mu2>
-    <kp>1000000.0</kp>
-    <kd>100.0</kd>
-  </gazebo>
-  <gazebo reference="wheel_rear_right_link">
-    <material>Gazebo/Black</material>
-    <mu1>1.0</mu1>
-    <mu2>1.0</mu2>
-    <kp>1000000.0</kp>
-    <kd>100.0</kd>
-  </gazebo>
-</robot>
+/home/xkai/agribot/agribot_ws/src/diff_drive_robot/urdf/robot.gazebo.xacro

File: agribot_ws/install/diff_drive_robot/share/diff_drive_robot/urdf/robot.urdf.xacro (robot description, xacro)
@@ -1,106 +1 @@
-<?xml version="1.0"?>
-<robot xmlns:xacro="http://www.ros.org/wiki/xacro" name="diff_drive_robot">
-  <!-- Import materials -->
-  <xacro:include filename="$(find diff_drive_robot)/urdf/materials.xacro"/>
-  <!-- Import Gazebo configurations -->
-  <xacro:include filename="$(find diff_drive_robot)/urdf/robot.gazebo.xacro"/>
-  <!-- Import IMU sensor -->
-  <xacro:include filename="$(find agribot_simulation)/urdf/agribot/sensors/imu.urdf.xacro" />
-  <!-- Import mid360 lidar -->
-  <xacro:include filename="$(find ros2_livox_simulation)/urdf/mid360.xacro" />
-  <!-- Robot dimensions (synchronized with agribot_simulation) -->
-  <xacro:property name="chassis_length" value="0.25"/>
-  <xacro:property name="chassis_width" value="0.20"/>
-  <xacro:property name="chassis_height" value="0.08"/>
-  <xacro:property name="chassis_mass" value="2.5"/>
-  <xacro:property name="wheel_radius" value="0.032"/>
-  <xacro:property name="wheel_thickness" value="0.02"/>
-  <xacro:property name="wheel_mass" value="0.2"/>
-  <!-- Wheel positions (from agribot_simulation) -->
-  <xacro:property name="wheel_offset_x_front" value="0.0789"/>
-  <xacro:property name="wheel_offset_x_rear" value="0.0930"/>
-  <xacro:property name="wheel_offset_y_left" value="0.0909"/>
-  <xacro:property name="wheel_offset_y_right" value="0.0907"/>
-  <xacro:property name="wheel_offset_z" value="-0.0363"/>
-  <!-- Base footprint link (ground projection) -->
-  <link name="base_footprint"/>
-  <!-- Joint from base_footprint to base_link -->
-  <joint name="base_joint" type="fixed">
-    <parent link="base_footprint"/>
-    <child link="base_link"/>
-    <origin xyz="0 0 ${wheel_radius - wheel_offset_z}" rpy="0 0 0"/>
-  </joint>
-  <!-- Base link (chassis) -->
-  <link name="base_link">
-    <visual>
-      <geometry>
-        <mesh filename="file://$(find agribot_simulation)/urdf/meshes/mini_4wd_robot_meshes/base_link.STL"/>
-      </geometry>
-      <material name="chassis_blue"/>
-      <origin xyz="0 0 0" rpy="0 0 0"/>
-    </visual>
-    <collision>
-      <geometry>
-        <box size="${chassis_length} ${chassis_width} ${chassis_height}"/>
-      </geometry>
-      <origin xyz="0 0 0" rpy="0 0 0"/>
-    </collision>
-    <inertial>
-      <mass value="${chassis_mass}"/>
-      <origin xyz="0 0 0" rpy="0 0 0"/>
-      <inertia
-        ixx="${chassis_mass / 12.0 * (chassis_width * chassis_width + chassis_height * chassis_height)}"
-        ixy="0.0"
-        ixz="0.0"
-        iyy="${chassis_mass / 12.0 * (chassis_length * chassis_length + chassis_height * chassis_height)}"
-        iyz="0.0"
-        izz="${chassis_mass / 12.0 * (chassis_length * chassis_length + chassis_width * chassis_width)}"/>
-    </inertial>
-  </link>
-  <!-- Macro for creating wheels -->
-  <xacro:macro name="wheel" params="prefix x_reflect y_reflect x_offset y_offset agribot_prefix">
-    <link name="wheel_${prefix}_link">
-      <visual>
-        <geometry>
-          <mesh filename="file://$(find agribot_simulation)/urdf/meshes/mini_4wd_robot_meshes/${agribot_prefix}_wheel_link.STL"/>
-        </geometry>
-        <material name="wheel_black"/>
-        <origin xyz="0 0 0" rpy="0 0 0"/>
-      </visual>
-      <collision>
-        <geometry>
-          <cylinder radius="${wheel_radius}" length="${wheel_thickness}"/>
-        </geometry>
-        <origin xyz="0 0 0" rpy="${pi / 2.0} 0 0"/>
-      </collision>
-      <inertial>
-        <mass value="${wheel_mass}"/>
-        <origin xyz="0 0 0" rpy="0 0 0"/>
-        <inertia
-          ixx="${wheel_mass / 12.0 * (3 * wheel_radius * wheel_radius + wheel_thickness * wheel_thickness)}"
-          ixy="0.0"
-          ixz="0.0"
-          iyy="${wheel_mass * wheel_radius * wheel_radius / 2.0}"
-          iyz="0.0"
-          izz="${wheel_mass / 12.0 * (3 * wheel_radius * wheel_radius + wheel_thickness * wheel_thickness)}"/>
-      </inertial>
-    </link>
-    <joint name="wheel_${prefix}_joint" type="continuous">
-      <parent link="base_link"/>
-      <child link="wheel_${prefix}_link"/>
-      <origin xyz="${x_reflect * x_offset} ${y_reflect * y_offset} ${wheel_offset_z}" rpy="0 0 0"/>
-      <axis xyz="0 1 0"/>
-    </joint>
-  </xacro:macro>
-  <!-- Create four wheels -->
-  <xacro:wheel prefix="front_left" x_reflect="1" y_reflect="1" x_offset="${wheel_offset_x_front}" y_offset="${wheel_offset_y_left}" agribot_prefix="lf"/>
-  <xacro:wheel prefix="rear_left" x_reflect="-1" y_reflect="1" x_offset="${wheel_offset_x_rear}" y_offset="${wheel_offset_y_left}" agribot_prefix="lb"/>
-  <xacro:wheel prefix="front_right" x_reflect="1" y_reflect="-1" x_offset="${wheel_offset_x_front}" y_offset="${wheel_offset_y_right}" agribot_prefix="rf"/>
-  <xacro:wheel prefix="rear_right" x_reflect="-1" y_reflect="-1" x_offset="${wheel_offset_x_rear}" y_offset="${wheel_offset_y_right}" agribot_prefix="rb"/>
-  <!-- IMU sensor -->
-  <xacro:imu_xacro xyz="0 0 0" />
-  <!-- mid360 lidar -->
-  <xacro:mid360 name="livox" parent="base_link" topic="mid360">
-    <origin xyz="0.1 0 0.1" rpy="0 0 0" />
-  </xacro:mid360>
-</robot>
+/home/xkai/agribot/agribot_ws/src/diff_drive_robot/urdf/robot.urdf.xacro
